Commit message: fix v3 (groudingDino) (enfin fonctionnelle), fin finetuning v1.1.1, fix objet flottant, ajout table

File: objets/001_table/table.urdf (robot description, URDF)
Before this commit: robot table, 5 links, 4 joints
Links:
- removed link table
- added link base
- added link tabletop; collision mesh filename=tabletop.obj; visual mesh filename=tabletop.obj
- link leg_bl: mass 1.0 -> None; geometry collision mesh filename=leg.obj; visual mesh filename=leg.obj
- link leg_br: mass 1.0 -> None; geometry collision mesh filename=leg.obj; visual mesh filename=leg.obj
- link leg_fl: mass 1.0 -> None; geometry collision mesh filename=leg.obj; visual mesh filename=leg.obj
- link leg_fr: mass 1.0 -> None; geometry collision mesh filename=leg.obj; visual mesh filename=leg.obj
Joints:
- added joint joint_tabletop: type fixed, parent base, child tabletop, origin xyz=0 0 0.725
- joint joint_leg_bl: origin xyz=-0.45 0.25 -0.375 rpy=0 0 0 -> xyz=-0.55 -0.35 0.35; parent table -> base
- joint joint_leg_br: origin xyz=-0.45 -0.25 -0.375 rpy=0 0 0 -> xyz=-0.55 0.35 0.35; parent table -> base
- joint joint_leg_fl: origin xyz=0.45 0.25 -0.375 rpy=0 0 0 -> xyz=0.55 -0.35 0.35; parent table -> base
- joint joint_leg_fr: origin xyz=0.45 -0.25 -0.375 rpy=0 0 0 -> xyz=0.55 0.35 0.35; parent table -> base
