Commit message: images formualires + autres stuff + objets renomés.

File: objets/ycb_mug.urdf (robot description, URDF)
Before this commit: robot 025_mug, 1 links, 0 joints
Links:
- link _name: geometry collision mesh filename=mug/google_16k/textured_vhacd.obj scale=1 1 1; visual mesh filename=mug/google_16k/textured.obj scale=1 1 1
